File: Dash4.brd (EAGLE design)
At the start: 100 x 26.7 mm, 9 parts

Commit message: Added GPIO pinout drawing, cleaned up schematic
Parts:
- removed LED1: (no value), adafruit:LED5MM
- removed R2: 330, adafruit:0207/9
Connections:
- removed net N$8: LED1.K, R2.2
- net N$2: no longer LED1.A
- net N$5: no longer R2.1
Routing:
- net N$7: track 92.4 -> 19.4 mm
- net N$2: track 26.0 -> 18.8 mm
Changed lines of the file:
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@@
 <attribute name="VALUE" x="58.42" y="15.875" size="1.27" layer="27" align="top-center"/>
-</element>
-<element name="LED1" library="adafruit" library_urn="urn:adsk.eagle:library:420" package="LED5MM" package3d_urn="urn:adsk.eagle:package:6240538/1" value="" x="3.81" y="-3.81" smashed="yes">
-<attribute name="NAME" x="6.985" y="-3.2766" size="1.27" layer="25" ratio="10"/>
-<attribute name="VALUE" x="7.0104" y="-5.6134" size="1.27" layer="27" ratio="10"/>
-</element>
-<element name="R2" library="adafruit" package="0207/9" value="330" x="6.35" y="-11.43" smashed="yes">
-<attribute name="NAME" x="3.302" y="-9.906" size="1.27" layer="25" ratio="10"/>
-<attribute name="VALUE" x="4.0894" y="-12.065" size="1.27" layer="27" ratio="10"/>
 </element>
 </elements>
@@
 <contactref element="U$1" pad="D2"/>
 <contactref element="U$1" pad="B2"/>
-<contactref element="U$2" pad="BAT+"/>
-<wire x1="31.75" y1="3.81" x2="26.67" y2="8.89" width="0.1524" layer="16"/>
 <wire x1="26.67" y1="8.89" x2="25.4" y2="10.16" width="0.1524" layer="16"/>
 <wire x1="26.67" y1="13.97" x2="25.4" y2="15.24" width="0.1524" layer="16"/>
@@
 <wire x1="25.4" y1="10.16" x2="24.765" y2="10.16" width="0.1524" layer="1"/>
 <wire x1="17.78" y1="6.985" x2="17.78" y2="6.858" width="0.1524" layer="1"/>
-<contactref element="LED1" pad="A"/>
-<wire x1="2.54" y1="-3.81" x2="17.78" y2="6.858" width="0" layer="19" extent="1-1"/>
+<contactref element="U$2" pad="BAT+"/>
+<wire x1="26.67" y1="8.89" x2="31.75" y2="3.81" width="0" layer="19" extent="16-16"/>
 </signal>
 <signal name="N$3">
@@
 <wire x1="93.6625" y1="13.97" x2="88.5825" y2="8.89" width="0.1524" layer="1"/>
 <wire x1="97.23" y1="13.97" x2="93.6625" y2="13.97" width="0.1524" layer="1"/>
-<contactref element="R2" pad="1"/>
-<wire x1="1.778" y1="-11.43" x2="22.86" y2="10.16" width="0" layer="19" extent="1-1"/>
 </signal>
 <signal name="N$6">
@@
 </signal>
 <signal name="N$7">
-<contactref element="U$2" pad="BAT-"/>
 <contactref element="SW3" pad="P$1"/>
 <contactref element="SW2" pad="P$1"/>
@@
 <wire x1="90.805" y1="8.89" x2="90.73" y2="8.89" width="0.1524" layer="16"/>
 <wire x1="90.805" y1="13.97" x2="90.73" y2="13.97" width="0.1524" layer="16"/>
-<wire x1="24.13" y1="15.5575" x2="24.13" y2="8.89" width="0.1524" layer="16"/>
-<wire x1="30.1625" y1="21.59" x2="24.13" y2="15.5575" width="0.1524" layer="16"/>
-<wire x1="31.75" y1="21.59" x2="30.1625" y2="21.59" width="0.1524" layer="16"/>
 <wire x1="87.9475" y1="21.59" x2="90.4875" y2="19.05" width="0.1524" layer="1"/>
-<wire x1="31.75" y1="21.59" x2="87.9475" y2="21.59" width="0.1524" layer="1"/>
 <wire x1="90.4875" y1="19.05" x2="90.73" y2="19.05" width="0.1524" layer="1"/>
+<contactref element="U$2" pad="BAT-"/>
 <contactref element="U$1" pad="A1"/>
-<wire x1="22.86" y1="7.62" x2="24.13" y2="8.89" width="0" layer="19" extent="16-16"/>
-</signal>
-<signal name="N$8">
-<contactref element="R2" pad="2"/>
-<contactref element="LED1" pad="K"/>
-<wire x1="10.922" y1="-11.43" x2="5.08" y2="-3.81" width="0" layer="19" extent="1-1"/>
+<wire x1="31.75" y1="21.59" x2="87.9475" y2="21.59" width="0" layer="19" extent="1-1"/>
+<wire x1="22.86" y1="7.62" x2="31.75" y2="21.59" width="0" layer="19" extent="1-1"/>
 </signal>
 </signals>
