File: CurrentSensor.sch (EAGLE design)
At the start: 20 parts, among them T1 2N3904, T2 2N3904, T3 2N3904, T4 2N3904

Commit message: Add files via upload
Parts:
- removed SW1, SW2, SW3, SW4: (no value), adafruit:SWITCH_PUSHBUTTONEVQ-PE
- removed U$1: WIRELESS-WIFI-ESP-01, diy-modules:WIRELESS-WIFI-ESP-01
- removed U$2: BATTERY-HOLDER-2AAA, diy-modules:BATTERY-HOLDER-2AAA
- added ESP8266-01: WIRELESS-WIFI-ESP-01, diy-modules:WIRELESS-WIFI-ESP-01
- added R7: 10k, adafruit:R-US_0207/9
- C1: value (none) -> 10uf
- JP1: value (none) -> Sensor
- R2: value 10k -> 1m
- R4: value 10k -> 220
- R5: value 10k -> 4K7
Connections:
- removed net N$1: SW4.P$2
- removed net N$2: U$2.BAT+
- removed net N$4: SW1.P$2
- removed net N$6: SW3.P$2
- removed net N$7: SW1.P$1, SW2.P$1, SW3.P$1, SW4.P$1, U$2.BAT-
- new net /OUT: ESP8266-01.GPIO2, R6.2, T4.C
- new net 3V3: ESP8266-01.CH_PD, ESP8266-01.VCC, R2.1, R3.1, R4.1, R6.1, R7.1
- new net N$17: ESP8266-01.RST, R7.2
- net GND: now also ESP8266-01.GND, R5.2; no longer R1.2
- net N$10: now also R5.1; no longer R1.1
- net N$13: now also R3.2; no longer R5.2
- net N$14: now also R2.2; no longer R6.2
- net N$15: now also R1.2; no longer R3.2
- net N$3: now also R1.1; no longer R3.1
Other:
- note added: "Current Sensor"
- note added: "Notes: R1 determines the sensitivity. Can be 0Ω R4 controls the intensity of the LED. Can be 0Ω"
- note removed: "Eight function DASH button"
- moved on the sheet: C1, D1, JP1, LED1, R1, R2, R3, R4, R5, R6, T1, T2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

Commit message: Add files via upload
Added an on-board regulator.
Parts:
- removed ESP8266-01: WIRELESS-WIFI-ESP-01, diy-modules:WIRELESS-WIFI-ESP-01
- added ESP-01: WIRELESS-WIFI-ESP-01, myParts:WIRELESS-WIFI-ESP-01
- added JP2: Gnd, adafruit:PINHD-1X1
- added JP3: 3V3, adafruit:PINHD-1X1CB
- added JP4: Vin, adafruit:PINHD-1X1CB
- added JP5: Gnd, adafruit:PINHD-1X1CB
- added PSU: In Out Gnd, adafruit:PINHD-1X3CB
- C1: device adafruit:C-US025-040X050 -> adafruit:CPOL-USE15-5AXIAL
Connections:
- new net N$1: JP4.1, PSU.1
- net /OUT: now also ESP-01.GPIO2; no longer ESP8266-01.GPIO2
- net 3V3: now also ESP-01.CH_PD, ESP-01.VCC, JP3.1, PSU.2; no longer ESP8266-01.CH_PD, ESP8266-01.VCC
- net GND: now also C1.-, ESP-01.GND, JP2.1, JP5.1, PSU.3; no longer C1.2, ESP8266-01.GND
- net N$10: now also C1.+; no longer C1.1
- net N$17: now also ESP-01.RST; no longer ESP8266-01.RST
Changed lines of the file:
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@@
 </classes>
 <parts>
-<part name="ESP8266-01" library="diy-modules" deviceset="WIRELESS-WIFI-ESP-01" device=""/>
 <part name="R5" library="adafruit" deviceset="R-US_" device="0207/9" value="4K7"/>
 <part name="FRAME1" library="frames" library_urn="urn:adsk.eagle:library:229" deviceset="LETTER_L" device=""/>
@@
 <part name="LED1" library="adafruit" library_urn="urn:adsk.eagle:library:420" deviceset="LED" device="5MM" package3d_urn="urn:adsk.eagle:package:6240538/1"/>
 <part name="D1" library="diode" library_urn="urn:adsk.eagle:library:210" deviceset="1N4148" device="DO35-10" package3d_urn="urn:adsk.eagle:package:43344/2" value="1N4148"/>
-<part name="C1" library="adafruit" deviceset="C-US" device="025-040X050" value="10uf"/>
 <part name="JP1" library="adafruit" library_urn="urn:adsk.eagle:library:420" deviceset="PINHD-1X1" device="" package3d_urn="urn:adsk.eagle:package:6240654/1" value="Sensor"/>
 <part name="T1" library="transistor" library_urn="urn:adsk.eagle:library:402" deviceset="2N3904" device="" package3d_urn="urn:adsk.eagle:package:28523/2"/>
@@
 <part name="R2" library="adafruit" deviceset="R-US_" device="0207/9" value="1m"/>
 <part name="R6" library="adafruit" deviceset="R-US_" device="0207/9" value="10k"/>
+<part name="SUPPLY2" library="supply2" library_urn="urn:adsk.eagle:library:372" deviceset="GND" device=""/>
+<part name="PSU" library="adafruit" library_urn="urn:adsk.eagle:library:420" deviceset="PINHD-1X3" device="CB" package3d_urn="urn:adsk.eagle:package:6240706/1" value="In Out Gnd"/>
+<part name="JP3" library="adafruit" deviceset="PINHD-1X1" device="CB" value="3V3"/>
+<part name="JP4" library="adafruit" deviceset="PINHD-1X1" device="CB" value="Vin"/>
+<part name="JP5" library="adafruit" deviceset="PINHD-1X1" device="CB" value="Gnd"/>
+<part name="C1" library="adafruit" library_urn="urn:adsk.eagle:library:420" deviceset="CPOL-US" device="E15-5AXIAL" package3d_urn="urn:adsk.eagle:package:6240491/1" value="10uf"/>
+<part name="ESP-01" library="myParts" deviceset="WIRELESS-WIFI-ESP-01" device=""/>
+<part name="JP2" library="adafruit" library_urn="urn:adsk.eagle:library:420" deviceset="PINHD-1X1" device="" package3d_urn="urn:adsk.eagle:package:6240654/1" value="Gnd"/>
+<part name="SUPPLY6" library="supply2" library_urn="urn:adsk.eagle:library:372" deviceset="GND" device=""/>
 </parts>
 <sheets>
@@
 </plain>
 <instances>
-<instance part="ESP8266-01" gate="G$1" x="193.04" y="104.14" smashed="yes">
-<attribute name="NAME" x="182.118" y="117.602" size="1.778" layer="95"/>
-</instance>
 <instance part="R5" gate="G$1" x="109.22" y="78.74" smashed="yes" rot="R270">
 <attribute name="NAME" x="110.4646" y="75.184" size="1.778" layer="95" rot="R270"/>
@@
 <attribute name="DRAWING_NAME" x="165.1" y="19.05" size="2.54" layer="94"/>
 </instance>
-<instance part="FRAME2" gate="G$1" x="0" y="0" smashed="yes"/>
 <instance part="FRAME2" gate="G$2" x="147.32" y="0" smashed="yes">
 <attribute name="LAST_DATE_TIME" x="160.02" y="1.27" size="2.54" layer="94"/>
@@
 <attribute name="VALUE" x="99.568" y="88.3666" size="1.778" layer="96"/>
 </instance>
-<instance part="C1" gate="G$1" x="101.6" y="81.28" smashed="yes">
-<attribute name="NAME" x="90.932" y="77.089" size="1.778" layer="95"/>
-<attribute name="VALUE" x="96.012" y="77.089" size="1.778" layer="96"/>
-</instance>
 <instance part="JP1" gate="G$1" x="50.8" y="109.22" smashed="yes" rot="R180">
 <attribute name="NAME" x="57.15" y="106.045" size="1.778" layer="95" rot="R180"/>
@@
 <attribute name="NAME" x="120.6246" y="123.444" size="1.778" layer="95" rot="R270"/>
 <attribute name="VALUE" x="120.65" y="129.032" size="1.778" layer="96" rot="R270"/>
+</instance>
+<instance part="SUPPLY2" gate="GND" x="195.58" y="129.54" smashed="yes">
+<attribute name="VALUE" x="193.675" y="126.365" size="1.778" layer="96"/>
+</instance>
+<instance part="PSU" gate="A" x="193.04" y="147.32" smashed="yes" rot="R90">
+<attribute name="NAME" x="187.325" y="140.97" size="1.778" layer="95" rot="R90"/>
+<attribute name="VALUE" x="200.66" y="140.97" size="1.778" layer="96" rot="R90"/>
+</instance>
+<instance part="JP3" gate="G$1" x="160.02" y="157.48" smashed="yes" rot="R90">
+<attribute name="NAME" x="156.845" y="151.13" size="1.778" layer="95" rot="R90"/>
+<attribute name="VALUE" x="165.1" y="151.13" size="1.778" layer="96" rot="R90"/>
+</instance>
+<instance part="JP4" gate="G$1" x="175.26" y="157.48" smashed="yes" rot="R90">
+<attribute name="NAME" x="172.085" y="151.13" size="1.778" layer="95" rot="R90"/>
+<attribute name="VALUE" x="180.34" y="151.13" size="1.778" layer="96" rot="R90"/>
+</instance>
+<instance part="JP5" gate="G$1" x="208.28" y="157.48" smashed="yes" rot="R90">
+<attribute name="NAME" x="205.105" y="151.13" size="1.778" layer="95" rot="R90"/>
+<attribute name="VALUE" x="213.36" y="151.13" size="1.778" layer="96" rot="R90"/>
+</instance>
+<instance part="C1" gate="G$1" x="101.6" y="81.28" smashed="yes">
+<attribute name="NAME" x="96.012" y="81.407" size="1.778" layer="95" rot="R180"/>
+<attribute name="VALUE" x="92.456" y="77.089" size="1.778" layer="96"/>
+</instance>
+<instance part="ESP-01" gate="G$1" x="177.8" y="106.68" smashed="yes">
+<attribute name="NAME" x="175.26" y="121.92" size="1.778" layer="95"/>
+<attribute name="VALUE" x="175.26" y="119.38" size="1.778" layer="96"/>
+</instance>
+<instance part="JP2" gate="G$1" x="50.8" y="96.52" smashed="yes" rot="R180">
+<attribute name="NAME" x="57.15" y="93.345" size="1.778" layer="95" rot="R180"/>
+<attribute name="VALUE" x="57.15" y="101.6" size="1.778" layer="96" rot="R180"/>
+</instance>
+<instance part="SUPPLY6" gate="GND" x="60.96" y="91.44" smashed="yes">
+<attribute name="VALUE" x="59.055" y="88.265" size="1.778" layer="96"/>
 </instance>
 </instances>
@@
 <wire x1="109.22" y1="83.82" x2="109.22" y2="86.36" width="0.1524" layer="91"/>
 <junction x="109.22" y="86.36"/>
-<pinref part="C1" gate="G$1" pin="1"/>
 <wire x1="101.6" y1="83.82" x2="101.6" y2="86.36" width="0.1524" layer="91"/>
 <junction x="101.6" y="86.36"/>
+<pinref part="C1" gate="G$1" pin="+"/>
 </segment>
 </net>
 <net name="GND" class="0">
 <segment>
-<pinref part="C1" gate="G$1" pin="2"/>
 <pinref part="SUPPLY1" gate="GND" pin="GND"/>
 <wire x1="101.6" y1="76.2" x2="101.6" y2="71.12" width="0.1524" layer="91"/>
+<pinref part="C1" gate="G$1" pin="-"/>
 </segment>
 <segment>
@@
 </segment>
 <segment>
-<pinref part="ESP8266-01" gate="G$1" pin="GND"/>
 <pinref part="SUPPLY5" gate="GND" pin="GND"/>
 <wire x1="170.18" y1="114.3" x2="144.78" y2="114.3" width="0.1524" layer="91"/>
 <wire x1="144.78" y1="114.3" x2="144.78" y2="71.12" width="0.1524" layer="91"/>
+<pinref part="ESP-01" gate="G$1" pin="GND"/>
+</segment>
+<segment>
+<pinref part="SUPPLY2" gate="GND" pin="GND"/>
+<wire x1="195.58" y1="132.08" x2="195.58" y2="137.16" width="0.1524" layer="91"/>
+<wire x1="195.58" y1="137.16" x2="195.58" y2="144.78" width="0.1524" layer="91"/>
+<wire x1="195.58" y1="137.16" x2="208.28" y2="137.16" width="0.1524" layer="91"/>
+<junction x="195.58" y="137.16"/>
+<wire x1="208.28" y1="137.16" x2="208.28" y2="154.94" width="0.1524" layer="91"/>
+<pinref part="PSU" gate="A" pin="3"/>
+<pinref part="JP5" gate="G$1" pin="1"/>
+</segment>
+<segment>
+<pinref part="JP2" gate="G$1" pin="1"/>
+<wire x1="53.34" y1="96.52" x2="60.96" y2="96.52" width="0.1524" layer="91"/>
+<pinref part="SUPPLY6" gate="GND" pin="GND"/>
+<wire x1="60.96" y1="96.52" x2="60.96" y2="93.98" width="0.1524" layer="91"/>
 </segment>
 </net>
@@
 <pinref part="R6" gate="G$1" pin="2"/>
 <wire x1="119.38" y1="91.44" x2="119.38" y2="109.22" width="0.1524" layer="91"/>
-<pinref part="ESP8266-01" gate="G$1" pin="GPIO2"/>
 <wire x1="119.38" y1="109.22" x2="119.38" y2="121.92" width="0.1524" layer="91"/>
 <wire x1="170.18" y1="109.22" x2="119.38" y2="109.22" width="0.1524" layer="91"/>
 <junction x="119.38" y="109.22"/>
 <label x="121.158" y="110.49" size="1.778" layer="95"/>
+<pinref part="ESP-01" gate="G$1" pin="GPIO2"/>
 </segment>
 </net>
@@
 <wire x1="119.38" y1="134.62" x2="139.7" y2="134.62" width="0.1524" layer="91"/>
 <wire x1="139.7" y1="134.62" x2="139.7" y2="96.52" width="0.1524" layer="91"/>
-<pinref part="ESP8266-01" gate="G$1" pin="VCC"/>
 <wire x1="139.7" y1="96.52" x2="152.4" y2="96.52" width="0.1524" layer="91"/>
 <pinref part="R6" gate="G$1" pin="1"/>
@@
 <wire x1="152.4" y1="101.6" x2="152.4" y2="96.52" width="0.1524" layer="91"/>
 <junction x="152.4" y="96.52"/>
-<pinref part="ESP8266-01" gate="G$1" pin="CH_PD"/>
 <wire x1="170.18" y1="106.68" x2="152.4" y2="106.68" width="0.1524" layer="91"/>
 <wire x1="152.4" y1="106.68" x2="152.4" y2="101.6" width="0.1524" layer="91"/>
 <junction x="152.4" y="101.6"/>
+<wire x1="139.7" y1="134.62" x2="160.02" y2="134.62" width="0.1524" layer="91"/>
+<junction x="139.7" y="134.62"/>
+<wire x1="160.02" y1="134.62" x2="193.04" y2="134.62" width="0.1524" layer="91"/>
+<wire x1="193.04" y1="134.62" x2="193.04" y2="144.78" width="0.1524" layer="91"/>
+<pinref part="PSU" gate="A" pin="2"/>
+<pinref part="JP3" gate="G$1" pin="1"/>
+<wire x1="160.02" y1="154.94" x2="160.02" y2="134.62" width="0.1524" layer="91"/>
+<junction x="160.02" y="134.62"/>
+<pinref part="ESP-01" gate="G$1" pin="CH_PD"/>
+<pinref part="ESP-01" gate="G$1" pin="VCC"/>
 </segment>
 </net>
@@
 <segment>
 <pinref part="R7" gate="G$1" pin="2"/>
-<pinref part="ESP8266-01" gate="G$1" pin="RST"/>
 <wire x1="165.1" y1="101.6" x2="170.18" y2="101.6" width="0.1524" layer="91"/>
-</segment>
-</net>
+<pinref part="ESP-01" gate="G$1" pin="RST"/>
+</segment>
+</net>
+<net name="N$1" class="0">
+<segment>
+<wire x1="190.5" y1="137.16" x2="190.5" y2="144.78" width="0.1524" layer="91"/>
+<pinref part="PSU" gate="A" pin="1"/>
+<pinref part="JP4" gate="G$1" pin="1"/>
+<wire x1="175.26" y1="154.94" x2="175.26" y2="137.16" width="0.1524" layer="91"/>
+<wire x1="175.26" y1="137.16" x2="190.5" y2="137.16" width="0.1524" layer="91"/>
+</segment>
+</net>
